File: power/power.kicad_pcb (KiCad board)
At the start: 2 copper layers, 24.1 x 31.8 mm, 12 parts, among them J1 PWR OFF, J2 VOUT, J3 GND, J4 VIN, J5 PWR BTN, Q1 Q_PMOS_GDS, Q2 Q_NMOS_GDS

Commit message: wip
Routing:
- net Net-(J5-Pad2): track 35.7 -> 42.2 mm
- net VCC: track 18.1 -> 22.1 mm
Other:
- board text added: "V2.0"
Changed lines of the file:
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@@
   (general
     (thickness 1.6)
-    (drawings 6)
-    (tracks 26)
+    (drawings 7)
+    (tracks 29)
     (zones 0)
     (modules 12)
@@
   (setup
     (last_trace_width 0.25)
+    (user_trace_width 2)
     (trace_clearance 0.2)
     (zone_clearance 0.508)
@@
       (effects (font (size 1 1) (thickness 0.15)))
     )
-    (fp_text user %R (at 0.3 0) (layer F.Fab)
-      (effects (font (size 1 1) (thickness 0.15)))
-    )
     (fp_circle (center 0 0) (end 2.2 0) (layer Cmts.User) (width 0.15))
     (fp_circle (center 0 0) (end 2.45 0) (layer F.CrtYd) (width 0.05))
+    (fp_text user %R (at 0.3 0) (layer F.Fab)
+      (effects (font (size 1 1) (thickness 0.15)))
+    )
     (pad 1 np_thru_hole circle (at 0 0) (size 2.2 2.2) (drill 2.2) (layers *.Cu *.Mask))
   )
@@
       (effects (font (size 1 1) (thickness 0.15)))
     )
-    (fp_text user %R (at 0.3 0) (layer F.Fab)
-      (effects (font (size 1 1) (thickness 0.15)))
-    )
     (fp_circle (center 0 0) (end 2.2 0) (layer Cmts.User) (width 0.15))
     (fp_circle (center 0 0) (end 2.45 0) (layer F.CrtYd) (width 0.05))
+    (fp_text user %R (at 0.3 0) (layer F.Fab)
+      (effects (font (size 1 1) (thickness 0.15)))
+    )
     (pad 1 np_thru_hole circle (at 0 0) (size 2.2 2.2) (drill 2.2) (layers *.Cu *.Mask))
   )
@@
     )
   )
+  (gr_text V2.0 (at 168.91 109.22) (layer F.SilkS)
+    (effects (font (size 1 1) (thickness 0.15)))
+  )
   (dimension 24.13 (width 0.15) (layer Dwgs.User)
     (gr_text "24,130 mm" (at 170.815 81.25) (layer Dwgs.User)
@@
   (gr_line (start 182.88 88.9) (end 182.88 120.65) (layer Edge.Cuts) (width 0.05))
   (segment (start 172.72 91.44) (end 177.8 91.44) (width 0.25) (layer F.Cu) (net 1))
-  (segment (start 166.42501 118.16501) (end 176.47499 118.16501) (width 2) (layer F.Cu) (net 2))
-  (segment (start 176.47499 118.16501) (end 179.07 115.57) (width 2) (layer F.Cu) (net 2))
-  (segment (start 165.1 116.84) (end 166.42501 118.16501) (width 0.25) (layer F.Cu) (net 2))
   (segment (start 179.07 115.57) (end 179.07 118.11) (width 2) (layer F.Cu) (net 2))
+  (segment (start 172.72 115.57) (end 179.07 115.57) (width 2) (layer F.Cu) (net 2))
+  (segment (start 171.45 119.38) (end 171.45 116.84) (width 2) (layer F.Cu) (net 2))
+  (segment (start 171.45 116.84) (end 172.72 115.57) (width 2) (layer F.Cu) (net 2))
+  (segment (start 165.1 119.38) (end 171.45 119.38) (width 2) (layer F.Cu) (net 2))
+  (segment (start 165.1 116.84) (end 165.1 119.38) (width 2) (layer F.Cu) (net 2))
   (segment (start 172.72 96.52) (end 177.8 96.52) (width 0.25) (layer F.Cu) (net 3))
   (segment (start 172.72 99.06) (end 167.64 104.14) (width 0.25) (layer F.Cu) (net 3))
@@
   (segment (start 172.72 99.06) (end 172.72 101.6) (width 0.25) (layer F.Cu) (net 3))
   (segment (start 177.8 96.52) (end 177.8 99.06) (width 0.25) (layer F.Cu) (net 3))
-  (segment (start 167.64 115.57) (end 173.99 109.22) (width 2) (layer F.Cu) (net 4))
-  (segment (start 167.64 116.84) (end 167.64 115.57) (width 0.25) (layer F.Cu) (net 4))
   (segment (start 173.99 109.22) (end 179.07 109.22) (width 2) (layer F.Cu) (net 4))
   (segment (start 179.07 109.22) (end 179.07 111.76) (width 2) (layer F.Cu) (net 4))
+  (segment (start 173.99 110.49) (end 167.64 116.84) (width 2) (layer F.Cu) (net 4))
+  (segment (start 173.99 109.22) (end 173.99 110.49) (width 2) (layer F.Cu) (net 4))
   (segment (start 166.42501 112.97499) (end 162.56 116.84) (width 0.25) (layer F.Cu) (net 5))
   (segment (start 166.42501 105.46501) (end 166.42501 112.97499) (width 0.25) (layer F.Cu) (net 5))
-  (segment (start 165.1 119.38) (end 173.99 119.38) (width 0.25) (layer F.Cu) (net 5))
-  (segment (start 162.56 116.84) (end 165.1 119.38) (width 0.25) (layer F.Cu) (net 5))
   (segment (start 173.140001 106.259999) (end 167.219999 106.259999) (width 0.25) (layer F.Cu) (net 5))
   (segment (start 173.99 105.41) (end 173.140001 106.259999) (width 0.25) (layer F.Cu) (net 5))
@@
   (segment (start 167.219999 106.259999) (end 166.37 105.41) (width 0.25) (layer F.Cu) (net 5))
   (segment (start 166.42501 105.46501) (end 166.37 105.41) (width 0.25) (layer F.Cu) (net 5))
+  (segment (start 162.56 116.84) (end 162.56 114.3) (width 0.25) (layer B.Cu) (net 5))
+  (segment (start 162.56 114.3) (end 173.99 114.3) (width 0.25) (layer B.Cu) (net 5))
+  (segment (start 173.99 114.3) (end 173.99 119.38) (width 0.25) (layer B.Cu) (net 5))
   (segment (start 162.56 91.44) (end 162.56 96.52) (width 0.25) (layer F.Cu) (net 6))
   (segment (start 162.56 96.52) (end 162.56 104.14) (width 0.25) (layer F.Cu) (net 6))
