File: pcb_control/power.kicad_sch (KiCad schematic)
At the start: 22 parts, among them J1 MCU_PWR, J19 FROM_MCU, J2 AUX_VOUT, J20 M_RGT, J21 BAT, J22 TO_MCU, J4 M_LFT, J5 PWR BTN, J6 MASTER_PWR_SW, Q1 Q_PMOS_GDS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

Commit message: wip
Parts:
- added NT2: NetTie_2, NetTie:NetTie-2_SMD_Pad2.0mm, symbol Device:NetTie_2
- C1: footprint Capacitor_THT:C_Axial_L12.0mm_D6.5mm_P15.00mm_Horizontal -> Capacitor_THT:C_Radial_D5.0mm_H11.0mm_P2.00mm
- J1: footprint (none) -> Connector_JST:JST_XH_B3B-XH-A_1x03_P2.50mm_Vertical
- J19, J22: footprint (none) -> Connector_JST:JST_XH_B6B-XH-A_1x06_P2.50mm_Vertical
- J2, J6: footprint (none) -> Connector_JST:JST_XH_B2B-XH-A_1x02_P2.50mm_Vertical
- J20, J4: footprint (none) -> Connector_JST:JST_XH_S6B-XH-A_1x06_P2.50mm_Horizontal
- J21: footprint (none) -> Connector_JST:JST_XH_S2B-XH-A-1_1x02_P2.50mm_Horizontal
- J5: footprint Connector_PinHeader_2.54mm:PinHeader_1x02_P2.54mm_Vertical -> Connector_JST:JST_XH_B2B-XH-A_1x02_P2.50mm_Vertical
- NT1: footprint (none) -> NetTie:NetTie-2_SMD_Pad2.0mm
- R5: value R33k -> 33k; footprint (none) -> Resistor_THT:R_Axial_DIN0207_L6.3mm_D2.5mm_P10.16mm_Horizontal
- R6: value R66k -> 66k; footprint (none) -> Resistor_THT:R_Axial_DIN0207_L6.3mm_D2.5mm_P10.16mm_Horizontal
- U2: footprint (none) -> tobi:drv8833
Connections:
- net +5V: no longer names the net of J1.2 (Pin_2), J20.2 (Pin_2), J4.2 (Pin_2), U1.1 (VOUT)
- net +BATT renamed XYZ
- net XYZ: no longer J21.2 (Pin_2), J6.1 (Pin_1), J6.2 (Pin_2), Q1.3 (S), R3.2, R5.1
- net GND renamed GND1
- net GND1: now also J21.2 (Pin_2); no longer J21.1 (Pin_1)
- net GND2: no longer names the net of J1.3 (Pin_3), NT1.2, U1.2 (GND)
- net GND2: now also NT2.1; no longer J20.5 (Pin_5), J4.5 (Pin_5)
- new net: J20.5 (Pin_5), J4.5 (Pin_5), NT2.2
- new net BAT1: J21.1 (Pin_1), J6.1 (Pin_1)
- new net BAT2: J6.2 (Pin_2), Q1.3 (S), R3.2, R5.1

Commit message: wip
Connections:
- net at Q2.1 (G), R1.1: no longer R2.2
- net at J1.1 (Pin_1), R1.2: now also R2.2
Other:
- moved on the sheet: R1
Changed lines of the file:
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@@
   (junction (at 64.516 69.723) (diameter 0) (color 0 0 0 0)
   )
+  (junction (at 77.216 116.078) (diameter 0) (color 0 0 0 0)
+  )
+  (junction (at 156.1592 113.538) (diameter 0) (color 0 0 0 0)
+  )
+  (junction (at 64.516 77.343) (diameter 0) (color 0 0 0 0)
+  )
+  (junction (at 58.166 116.078) (diameter 0) (color 0 0 0 0)
+  )
+  (junction (at 125.984 59.69) (diameter 0) (color 0 0 0 0)
+  )
+  (junction (at 64.516 69.596) (diameter 0) (color 0 0 0 0)
+  )
+  (junction (at 122.428 100.838) (diameter 0) (color 0 0 0 0)
+  )
   (junction (at 77.216 100.838) (diameter 0) (color 0 0 0 0)
-  )
-  (junction (at 77.216 116.078) (diameter 0) (color 0 0 0 0)
-  )
-  (junction (at 156.1592 113.538) (diameter 0) (color 0 0 0 0)
-  )
-  (junction (at 64.516 77.343) (diameter 0) (color 0 0 0 0)
-  )
-  (junction (at 58.166 116.078) (diameter 0) (color 0 0 0 0)
-  )
-  (junction (at 125.984 59.69) (diameter 0) (color 0 0 0 0)
-  )
-  (junction (at 64.516 69.596) (diameter 0) (color 0 0 0 0)
-  )
-  (junction (at 122.428 100.838) (diameter 0) (color 0 0 0 0)
   )
   (junction (at 118.491 60.706) (diameter 0) (color 0 0 0 0)
@@
     (stroke (width 0) (type default) (color 0 0 0 0))
   )
-  (wire (pts (xy 77.216 100.838) (xy 93.726 100.838))
-    (stroke (width 0) (type default) (color 0 0 0 0))
-  )
   (wire (pts (xy 155.829 50.673) (xy 155.829 67.31))
     (stroke (width 0) (type default) (color 0 0 0 0))
   )
+  (wire (pts (xy 77.216 100.838) (xy 81.5848 100.838))
+    (stroke (width 0) (type default) (color 0 0 0 0))
+  )
   (wire (pts (xy 155.829 67.31) (xy 181.356 67.31))
     (stroke (width 0) (type default) (color 0 0 0 0))
@@
     (stroke (width 0) (type default) (color 0 0 0 0))
   )
-  (wire (pts (xy 70.358 96.52) (xy 77.216 96.52))
-    (stroke (width 0) (type default) (color 0 0 0 0))
-  )
   (wire (pts (xy 31.242 87.884) (xy 31.242 90.678))
     (stroke (width 0) (type default) (color 0 0 0 0))
@@
     (stroke (width 0) (type default) (color 0 0 0 0))
   )
-  (wire (pts (xy 62.738 96.52) (xy 52.07 96.52))
-    (stroke (width 0) (type default) (color 0 0 0 0))
-  )
-  (wire (pts (xy 77.216 104.648) (xy 77.216 100.838))
-    (stroke (width 0) (type default) (color 0 0 0 0))
-  )
   (wire (pts (xy 107.442 53.086) (xy 83.82 53.086))
     (stroke (width 0) (type default) (color 0 0 0 0))
@@
     (stroke (width 0) (type default) (color 0 0 0 0))
   )
+  (wire (pts (xy 77.216 100.838) (xy 77.216 104.648))
+    (stroke (width 0) (type default) (color 0 0 0 0))
+  )
   (wire (pts (xy 132.207 113.538) (xy 143.129 113.538))
     (stroke (width 0) (type default) (color 0 0 0 0))
@@
     (stroke (width 0) (type default) (color 0 0 0 0))
   )
+  (wire (pts (xy 77.216 96.52) (xy 52.07 96.52))
+    (stroke (width 0) (type default) (color 0 0 0 0))
+  )
   (wire (pts (xy 100.076 90.678) (xy 98.806 90.678))
     (stroke (width 0) (type default) (color 0 0 0 0))
@@
     (stroke (width 0) (type default) (color 0 0 0 0))
   )
+  (wire (pts (xy 118.364 60.706) (xy 118.491 60.706))
+    (stroke (width 0) (type default) (color 0 0 0 0))
+  )
+  (wire (pts (xy 125.984 59.69) (xy 160.909 59.69))
+    (stroke (width 0) (type default) (color 0 0 0 0))
+  )
+  (wire (pts (xy 64.516 69.596) (xy 64.516 69.723))
+    (stroke (width 0) (type default) (color 0 0 0 0))
+  )
+  (wire (pts (xy 143.129 111.76) (xy 143.129 113.538))
+    (stroke (width 0) (type default) (color 0 0 0 0))
+  )
+  (wire (pts (xy 88.646 116.078) (xy 112.522 116.078))
+    (stroke (width 0) (type default) (color 0 0 0 0))
+  )
+  (wire (pts (xy 26.289 60.706) (xy 45.974 60.706))
+    (stroke (width 0) (type default) (color 0 0 0 0))
+  )
+  (wire (pts (xy 28.702 98.806) (xy 54.864 98.806))
+    (stroke (width 0) (type default) (color 0 0 0 0))
+  )
+  (wire (pts (xy 31.242 90.678) (xy 58.166 90.678))
+    (stroke (width 0) (type default) (color 0 0 0 0))
+  )
+  (wire (pts (xy 105.029 74.676) (xy 163.449 74.676))
+    (stroke (width 0) (type default) (color 0 0 0 0))
+  )
+  (wire (pts (xy 81.28 64.516) (xy 81.28 42.037))
+    (stroke (width 0) (type default) (color 0 0 0 0))
+  )
+  (wire (pts (xy 163.449 50.673) (xy 163.449 74.676))
+    (stroke (width 0) (type default) (color 0 0 0 0))
+  )
   (wire (pts (xy 77.216 96.52) (xy 77.216 100.838))
     (stroke (width 0) (type default) (color 0 0 0 0))
   )
-  (wire (pts (xy 118.364 60.706) (xy 118.491 60.706))
-    (stroke (width 0) (type default) (color 0 0 0 0))
-  )
-  (wire (pts (xy 125.984 59.69) (xy 160.909 59.69))
-    (stroke (width 0) (type default) (color 0 0 0 0))
-  )
-  (wire (pts (xy 64.516 69.596) (xy 64.516 69.723))
-    (stroke (width 0) (type default) (color 0 0 0 0))
-  )
-  (wire (pts (xy 143.129 111.76) (xy 143.129 113.538))
-    (stroke (width 0) (type default) (color 0 0 0 0))
-  )
-  (wire (pts (xy 88.646 116.078) (xy 112.522 116.078))
-    (stroke (width 0) (type default) (color 0 0 0 0))
-  )
-  (wire (pts (xy 26.289 60.706) (xy 45.974 60.706))
-    (stroke (width 0) (type default) (color 0 0 0 0))
-  )
-  (wire (pts (xy 28.702 98.806) (xy 54.864 98.806))
-    (stroke (width 0) (type default) (color 0 0 0 0))
-  )
-  (wire (pts (xy 31.242 90.678) (xy 58.166 90.678))
-    (stroke (width 0) (type default) (color 0 0 0 0))
-  )
-  (wire (pts (xy 105.029 74.676) (xy 163.449 74.676))
-    (stroke (width 0) (type default) (color 0 0 0 0))
-  )
-  (wire (pts (xy 81.28 64.516) (xy 81.28 42.037))
-    (stroke (width 0) (type default) (color 0 0 0 0))
-  )
-  (wire (pts (xy 163.449 50.673) (xy 163.449 74.676))
-    (stroke (width 0) (type default) (color 0 0 0 0))
-  )
   (wire (pts (xy 77.216 116.078) (xy 88.646 116.078))
     (stroke (width 0) (type default) (color 0 0 0 0))
@@
     (stroke (width 0) (type default) (color 0 0 0 0))
   )
+  (wire (pts (xy 89.2048 100.838) (xy 93.726 100.838))
+    (stroke (width 0) (type default) (color 0 0 0 0))
+  )
   (wire (pts (xy 105.029 69.596) (xy 128.524 69.596))
     (stroke (width 0) (type default) (color 0 0 0 0))
@@
     (effects (font (size 1.27 1.27)) (justify left bottom))
   )
-  (symbol (lib_id "Device:R") (at 66.548 96.52 270) (unit 1)
+  (symbol (lib_id "Device:R") (at 85.3948 100.838 270) (unit 1)
     (in_bom yes) (on_board yes)
-    (property "Reference" "R1" (id 0) (at 66.548 99.441 90))
-    (property "Value" "100" (id 1) (at 66.548 101.7524 90))
-    (property "Footprint" "Resistor_THT:R_Axial_DIN0207_L6.3mm_D2.5mm_P10.16mm_Horizontal" (id 2) (at 66.548 94.742 90)
-      (effects (font (size 1.27 1.27)) hide)
-    )
-    (property "Datasheet" "~" (id 3) (at 66.548 96.52 0)
+    (property "Reference" "R1" (id 0) (at 89.6366 99.2378 90))
+    (property "Value" "100" (id 1) (at 85.1662 98.5012 90))
+    (property "Footprint" "Resistor_THT:R_Axial_DIN0207_L6.3mm_D2.5mm_P10.16mm_Horizontal" (id 2) (at 85.3948 99.06 90)
+      (effects (font (size 1.27 1.27)) hide)
+    )
+    (property "Datasheet" "~" (id 3) (at 85.3948 100.838 0)
       (effects (font (size 1.27 1.27)) hide)
     )
@@
       (effects (font (size 1.27 1.27)) (justify left))
     )
-    (property "Value" "Q_NMOS_GDS" (id 1) (at 79.756 103.378 90)
+    (property "Value" "Q_NMOS_GDS" (id 1) (at 90.7034 111.887 90)
       (effects (font (size 1.27 1.27)) (justify left))
     )
